File: Celestine-PCB/Celestine.kicad_pcb (KiCad board)
At the start: 2 copper layers, 343.9 x 123.4 mm, 202 parts, among them SW1 SW_Push, U1 ATmega32U4-AU, U2 PRTR5V0U2X, Y1 16Mhz

Commit message: Update readme
Routing:
- net ROW2: track 357.8 -> 360.9 mm
- net ROW1: track 379.8 -> 383.0 mm
- net ROW3: track 287.4 -> 284.4 mm
- net ROW0: track 408.5 -> 411.1 mm

Commit message: Remove need for jumpers
Parts:
- removed JP1: UnifiedJumper, random-keyboard-parts:Jumper-UserFriendly
- removed JP2: SplitJumper, random-keyboard-parts:Jumper-UserFriendly
- removed REF**: H87A-Outline, locallib:H87A-Outline
- added G***: LOGO, locallib:ai-ring-6mm-Combined, F.Cu at (44.5, 101.6)
- added G***: LOGO, locallib:Celestine, F.Cu at (115.9, 64.3)
- added G***: LOGO, locallib:ai-ring-6mm-Combined, B.Cu at (73.8, 62.7)
- K_BACK1: footprint hitek725:Hitek725-2U -> hitek725:Hitek725-2U-DudPad
- K_SBACK2: footprint hitek725:Hitek725-1U -> hitek725:Hitek725-1U-DudPad
- moved U2 5.56 mm to (310.1, 9.37)
- moved USB1 5.56 mm to (310.1, -2.70)
- moved F1 4.76 mm to (307.2, 13.8)
- moved R73 4.55 mm to (301.6, 2.38), turned to 0 degrees
- moved R74 4.22 mm to (318.3, 2.38), turned to 180 degrees
Connections:
- K_BACK1 pad 1: FULLBACK -> Net-(D14-Pad2)
- K_SBACK1 pad 2: FULLBACK -> Net-(D14-Pad2)
- K_SBACK2 pad 2: FULLBACK -> Net-(D68-Pad2)
Routing:
- net FULLBACK: track 55.2 -> 0.00 mm
- net Net-(D14-Pad2): track 16.1 -> 55.7 mm
- net Net-(D68-Pad2): track 78.3 -> 62.3 mm, vias 2 -> 1
- net COL1: track 372.8 -> 358.7 mm
- net Net-(R68-Pad2): track 81.2 -> 76.3 mm
- net Net-(R67-Pad2): track 84.3 -> 79.4 mm
- net +5V: track 141.7 -> 137.0 mm
- net GND: track 235.9 -> 231.7 mm
- net Net-(R73-Pad2): track 8.50 -> 10.8 mm
- net Net-(R74-Pad2): track 8.66 -> 10.8 mm
- net VCC: track 18.4 -> 17.6 mm
Other:
- board size 343.9 x 123.4 mm -> 343.7 x 116.7 mm
- board text added: "Celestine TKL PCB Revision 1.0 20191110 | Credits to mcmaxmcmc, Engicoder for reverse engineering"
- board text added: "TKL PCB for NMB Hi-Tek 725 Switches"
- board text added: "www.ai03.me"
- board text removed: "Split"
- board text removed: "Unified"
