File: Celestine-PCB/Celestine.kicad_pcb (KiCad board)
At the start: 2 copper layers, 343.7 x 116.7 mm, 202 parts, among them SW1 SW_Push, U1 ATmega32U4-AU, U2 PRTR5V0U2X, Y1 16Mhz

Commit message: Progress
Parts:
- moved G*** 225.4 mm to (341.3, 67.5)
- moved G*** 5.61 mm to (38.9, 100.8)
- moved G*** 1.59 mm to (72.2, 62.7)
Routing:
- net COL14: track 130.0 -> 189.3 mm
- net COL15: track 141.6 -> 181.9 mm
- net ROW5: track 382.9 -> 373.8 mm
- net COL16: track 161.0 -> 166.4 mm
- net ROW3: track 284.4 -> 287.9 mm
- net ROW1: track 383.0 -> 379.8 mm
- net ROW2: track 360.9 -> 357.9 mm
- net COL1: track 358.7 -> 355.8 mm
- net ROW0: track 411.4 -> 408.5 mm
- net GND: track 231.7 -> 233.1 mm
- net COL0: track 394.6 -> 395.7 mm
- net Net-(R68-Pad2): track 76.3 -> 75.8 mm
Other:
- board text added: "Celestine TKL PCB Revision 1.1 20190413 | Credits to mcmaxmcmc, Engicoder for reverse engineering"
- board text added: "Hi-Tek 725 TKL"
- board text added: "kb.ai03.me"
- board text removed: "Celestine TKL PCB Revision 1.0 20191110 | Credits to mcmaxmcmc, Engicoder for reverse engineering"
- board text removed: "TKL PCB for NMB Hi-Tek 725 Switches"
- board text removed: "www.ai03.me"
