File: Celestine-PCB/Celestine.sch (KiCad schematic (older format))
At the start: 233 parts, among them Q1 2N7002, U1 ATmega32U4-MU, U2 PRTR5V0U2X, Y1 16Mhz

Commit message: Begin add libraries
Parts:
- removed U2: PRTR5V0U2X, locallib:SOT143B, symbol ai03-locallib:PRTR5V0U2X
- added U?: PRTR5V0U2X, symbol random-keyboard-parts:PRTR5V0U2X
- USB1: footprint Type-C:HRO-TYPE-C-31-M-12-Assembly -> (none)
Changed lines of the file:
@@
 EESchema Schematic File Version 4
+LIBS:Celestine-cache
 EELAYER 26 0
 EELAYER END
@@
 $EndComp
 $Comp
-L Type-C:HRO-TYPE-C-31-M-12 USB1
-U 1 1 5B361237
-P 1275 9100
-F 0 "USB1" H 1075 9750 60  0000 C CNN
-F 1 "HRO-TYPE-C-31-M-12" V 875 9050 60  0000 C CNN
-F 2 "Type-C:HRO-TYPE-C-31-M-12-Assembly" H 1275 9100 60  0001 C CNN
-F 3 "" H 1275 9100 60  0001 C CNN
-	1    1275 9100
-	1    0    0    -1
-$EndComp
-$Comp
 L power:GND #PWR015
 U 1 1 5B3665A1
@@
 	1    0    0    -1
 $EndComp
-$Comp
-L ai03-locallib:PRTR5V0U2X U2
-U 1 1 5C7DBF2D
-P 2975 9550
-F 0 "U2" H 2975 9847 60  0000 C CNN
-F 1 "PRTR5V0U2X" H 2975 9741 60  0000 C CNN
-F 2 "locallib:SOT143B" H 2975 9550 60  0001 C CNN
-F 3 "" H 2975 9550 60  0001 C CNN
-	1    2975 9550
-	1    0    0    -1
-$EndComp
 Wire Wire Line
 	3700 9175 4000 9175
@@
 	1    0    0    -1
 $EndComp
+$Comp
+L Type-C:HRO-TYPE-C-31-M-12 USB1
+U 1 1 5C3CCADA
+P 1275 9100
+F 0 "USB1" H 1106 9897 60  0000 C CNN
+F 1 "HRO-TYPE-C-31-M-12" H 1106 9791 60  0000 C CNN
+F 2 "" H 1275 9100 60  0001 C CNN
+F 3 "" H 1275 9100 60  0001 C CNN
+	1    1275 9100
+	1    0    0    -1
+$EndComp
+$Comp
+L random-keyboard-parts:PRTR5V0U2X U?
+U 1 1 5C3CD76D
+P 2975 9550
+F 0 "U?" H 2975 9847 60  0000 C CNN
+F 1 "PRTR5V0U2X" H 2975 9741 60  0000 C CNN
+F 2 "" H 2975 9550 60  0001 C CNN
+F 3 "" H 2975 9550 60  0001 C CNN
+	1    2975 9550
+	1    0    0    -1
+$EndComp

Commit message: Bind some footprints
Parts:
- U?: footprint (none) -> random-keyboard-parts:SOT143B
- USB1: footprint (none) -> Type-C:HRO-TYPE-C-31-M-12-Assembly
Changed lines of the file:
@@
 F 0 "USB1" H 1106 9897 60  0000 C CNN
 F 1 "HRO-TYPE-C-31-M-12" H 1106 9791 60  0000 C CNN
-F 2 "" H 1275 9100 60  0001 C CNN
+F 2 "Type-C:HRO-TYPE-C-31-M-12-Assembly" H 1275 9100 60  0001 C CNN
 F 3 "" H 1275 9100 60  0001 C CNN
 	1    1275 9100
@@
 F 0 "U?" H 2975 9847 60  0000 C CNN
 F 1 "PRTR5V0U2X" H 2975 9741 60  0000 C CNN
-F 2 "" H 2975 9550 60  0001 C CNN
+F 2 "random-keyboard-parts:SOT143B" H 2975 9550 60  0001 C CNN
 F 3 "" H 2975 9550 60  0001 C CNN
 	1    2975 9550

Commit message: Build generic schematic
Parts:
- removed D30, D58, D60, D62, D63: SOD-123, Diodes_SMD:D_SOD-123, symbol Device:D_Small
- removed K_RALT2, K_RMENU2, K_SPACE5: MX-1.25U, MX_Alps_Hybrid:MX-1.25U-FLIPPED, symbol MX_Alps_Hybrids:MX-1U
- removed K_RWIN3: MX-1U, MX_Alps_Hybrid:MX-1U, symbol MX_Alps_Hybrids:MX-1U
- removed K_SPACE3: MX-2.25U, MX_Alps_Hybrid:MX-2.25U-ReversedStabilizers, symbol MX_Alps_Hybrids:MX-1U
- removed K_SPACE4: MX-2.75U, MX_Alps_Hybrid:MX-2.75U-ReversedStabilizers, symbol MX_Alps_Hybrids:MX-1U
- removed K_WIN1: MX-1.25U, MX_Alps_Hybrid:MX-1.25U, symbol MX_Alps_Hybrids:MX-1U
- removed K_WIN2: MX-1U, MX_Alps_Hybrid:MX-1U-FLIPPED, symbol MX_Alps_Hybrids:MX-1U
- removed R30, R58, R60, R62, R63: 1k, Resistors_SMD:R_0805, symbol Device:R_Small
- K_ALT1: value MX-1.25U -> MX-1.5U; footprint MX_Alps_Hybrid:MX-1.25U -> MX_Alps_Hybrid:MX-1.5U
- K_CTRL1: value MX-1.25U -> MX-2U
- gave numbers to parts that had none: 2
Connections:
- wire segments 599 -> 600

Commit message: Build the PCB
Parts:
- removed D44, D57: SOD-123, Diodes_SMD:D_SOD-123, symbol Device:D_Small
- removed K_CAPS2: MX-1.25U, MX_Alps_Hybrid:MX-1.25U-FLIPPED, symbol MX_Alps_Hybrids:MX-1U
- removed K_SHIFT2: MX-1.25U, MX_Alps_Hybrid:MX-1.25U, symbol MX_Alps_Hybrids:MX-1U
- removed K_SHIFT3, K_SRSHIFT2, K_\2: MX-1U, MX_Alps_Hybrid:MX-1U, symbol MX_Alps_Hybrids:MX-1U
- removed K_SPACE2: MX-6.25U, MX_Alps_Hybrid:MX-6.25U-ReversedStabilizers, symbol MX_Alps_Hybrids:MX-1U
- removed K_SRSHIFT1: MX-1.75U, MX_Alps_Hybrid:MX-1.75U, symbol MX_Alps_Hybrids:MX-1U
- removed Q1: 2N7002, TO_SOT_Packages_SMD:SOT-23, symbol Transistor_FET:2N7002
- removed R1, R10, R11, R12, R13, R14, R16, R17, R18, R19, R2, R20, R21, R22, R23, R24, R25, R26, R27, R28, R29, R3, R31, R32, R33, R34, R35, R36, R37, R38, R39, R4, R40, R41, R42, R43, R44, R45, R46, R47, R48, R49, R5, R50, R51, R52, R53, R54, R55, R56, R57, R59, R6, R61, R64, R65, R69, R7, R72, R75, R8, R9: 1k, Resistors_SMD:R_0805, symbol Device:R_Small
- removed U1: ATmega32U4-MU, Housings_DFN_QFN:QFN-44-1EP_7x7mm_Pitch0.5mm, symbol MCU_Microchip_ATmega:ATmega32U4-MU
- added D15, D30, D58, D60, D62, D63, D66, D69, D70, D71, D72, D73, D74, D75, D76, D77, D78, D79, D80, D81, D82, D83, D84, D85, D86, D87, D88, D89: SOD-123, Diodes_SMD:D_SOD-123, symbol Device:D_Small
- added JP1: UnifiedJumper, random-keyboard-parts:Jumper-UserFriendly, symbol Device:Jumper_NO_Small
- added JP2: SplitJumper, random-keyboard-parts:Jumper-UserFriendly, symbol Device:Jumper_NO_Small
- added K_DEL1, K_DOWN1, K_END1, K_ESC1, K_FN1, K_FN10, K_FN11, K_FN12, K_FN2, K_FN3, K_FN4, K_FN5, K_FN6, K_FN7, K_FN8, K_FN9, K_HOME1, K_INS1, K_LEFT1, K_PAUSE1, K_PGDN1, K_PGUP1, K_PRTSC1, K_RIGHT1, K_RWIN1, K_SLCK1, K_UP1, K_WIN1: MX-1U, hitek725:Hitek725-1U, symbol MX_Alps_Hybrids:MX-1U
- added U1: ATmega32U4-AU, Housings_QFP:TQFP-44_10x10mm_Pitch0.8mm, symbol MCU_Microchip_ATmega:ATmega32U4-AU
- K_#1, K_#10, K_#2, K_#3, K_#4, K_#5, K_#6, K_#7, K_#8, K_#9, K_'1, K_,1, K_-1, K_.1, K_/1, K_;1, K_=1, K_A1, K_B1, K_C1, K_D1, K_E1, K_F1, K_G1, K_H1, K_I1, K_J1, K_K1, K_L1, K_M1, K_N1, K_O1, K_P1, K_Q1, K_R1, K_S1, K_SBACK1, K_SBACK2, K_T1, K_U1, K_V1, K_W1, K_X1, K_Y1, K_Z1, K_[1, K_]1: footprint MX_Alps_Hybrid:MX-1U -> hitek725:Hitek725-1U
- K_ALT1, K_TAB1, K_\1: footprint MX_Alps_Hybrid:MX-1.5U -> hitek725:Hitek725-1.5U
- K_ALT2, K_CTRL2: footprint MX_Alps_Hybrid:MX-1.5U-FLIPPED -> hitek725:Hitek725-1.5U
- K_BACK1: footprint MX_Alps_Hybrid:MX-2U -> hitek725:Hitek725-2U
- K_CAPS1: footprint MX_Alps_Hybrid:MX-1.75U -> hitek725:Hitek725-1.75U
- K_CTRL1: footprint MX_Alps_Hybrid:MX-1.25U -> hitek725:Hitek725-2U
- K_ENTER1, K_SHIFT1: footprint MX_Alps_Hybrid:MX-2.25U -> hitek725:Hitek725-2.25U
- K_ENTER2: value MX-ISO -> MX-BAE; footprint MX_Alps_Hybrid:MX-ISO-ReversedStabilizers -> hitek725:Hitek725-BigAssEnter-DudPad
- K_RALT1: renamed from K_RWIN2; value MX-1.25U -> MX-1.5U; footprint MX_Alps_Hybrid:MX-1.25U -> hitek725:Hitek725-1.5U
- K_RALT2: renamed from K_RALT3; footprint MX_Alps_Hybrid:MX-1.5U-FLIPPED -> hitek725:Hitek725-1.5U
- K_RCTRL1: renamed from K_RCTRL2; value MX-1.25U -> MX-2U; footprint MX_Alps_Hybrid:MX-1.25U -> hitek725:Hitek725-2U
- K_RCTRL2: renamed from K_RCTRL3; footprint MX_Alps_Hybrid:MX-1.5U-FLIPPED -> hitek725:Hitek725-1.5U
- K_RSHIFT1: footprint MX_Alps_Hybrid:MX-2.75U-FLIPPED -> hitek725:Hitek725-2.75U
- K_SPACE1: footprint MX_Alps_Hybrid:MX-7U-ReversedStabilizers -> hitek725:Hitek725-7U
- K_`1: renamed from K_ESC1; footprint MX_Alps_Hybrid:MX-1U -> hitek725:Hitek725-1U
- SW1: footprint (none) -> random-keyboard-parts:SKQG-1155865
Connections:
- net labels added: COL14, COL15, COL16, FULLBACK, ROW5, SPLITBACK
- net labels removed: LEDGND
- wire segments 600 -> 557

Commit message: Remove need for jumpers
Parts:
- removed JP1: UnifiedJumper, random-keyboard-parts:Jumper-UserFriendly, symbol Device:Jumper_NO_Small
- removed JP2: SplitJumper, random-keyboard-parts:Jumper-UserFriendly, symbol Device:Jumper_NO_Small
- K_BACK1: footprint hitek725:Hitek725-2U -> hitek725:Hitek725-2U-DudPad
- K_SBACK2: footprint hitek725:Hitek725-1U -> hitek725:Hitek725-1U-DudPad
Connections:
- net labels removed: FULLBACK, SPLITBACK
- wire segments 557 -> 548
Changed lines of the file:
@@
 F 0 "K_BACK1" H 9375 2875 60  0000 C CNN
 F 1 "MX-2U" H 9375 2800 20  0000 C CNN
-F 2 "hitek725:Hitek725-2U" H 9350 2725 60  0001 C CNN
+F 2 "hitek725:Hitek725-2U-DudPad" H 9350 2725 60  0001 C CNN
 F 3 "" H 9350 2725 60  0001 C CNN
 	1    9375 2750
@@
 L Device:D_Small D14
 U 1 1 5AC9C078
-P 10075 2850
-F 0 "D14" H 10025 2930 50  0000 L CNN
-F 1 "SOD-123" H 9975 3025 50  0000 L CNN
-F 2 "Diodes_SMD:D_SOD-123" V 10075 2850 50  0001 C CNN
-F 3 "" V 10075 2850 50  0001 C CNN
-	1    10075 2850
+P 9275 3025
+F 0 "D14" H 9225 3105 50  0000 L CNN
+F 1 "SOD-123" H 9175 3200 50  0000 L CNN
+F 2 "Diodes_SMD:D_SOD-123" V 9275 3025 50  0001 C CNN
+F 3 "" V 9275 3025 50  0001 C CNN
+	1    9275 3025
 	0    -1   -1   0
 $EndComp
@@
 F 0 "K_SBACK2" H 9375 4825 60  0000 C CNN
 F 1 "MX-1U" H 9375 4750 20  0000 C CNN
-F 2 "hitek725:Hitek725-1U" H 9350 4675 60  0001 C CNN
+F 2 "hitek725:Hitek725-1U-DudPad" H 9350 4675 60  0001 C CNN
 F 3 "" H 9350 4675 60  0001 C CNN
 	1    9375 4700
@@
 L Device:D_Small D68
 U 1 1 5B3729AC
-P 10350 2850
-F 0 "D68" H 10300 2930 50  0000 L CNN
-F 1 "SOD-123" H 10250 3025 50  0000 L CNN
-F 2 "Diodes_SMD:D_SOD-123" V 10350 2850 50  0001 C CNN
-F 3 "" V 10350 2850 50  0001 C CNN
-	1    10350 2850
+P 9275 4975
+F 0 "D68" H 9225 5055 50  0000 L CNN
+F 1 "SOD-123" H 9175 5150 50  0000 L CNN
+F 2 "Diodes_SMD:D_SOD-123" V 9275 4975 50  0001 C CNN
+F 3 "" V 9275 4975 50  0001 C CNN
+	1    9275 4975
 	0    -1   -1   0
 $EndComp
@@
 Wire Wire Line
 	9725 2575 9725 2925
-Text GLabel 9275 2925 3    50   Input ~ 0
-FULLBACK
-Text GLabel 9275 4875 3    50   Input ~ 0
-SPLITBACK
-Text GLabel 10150 2450 1    50   Input ~ 0
-FULLBACK
-Text GLabel 10250 2450 1    50   Input ~ 0
-SPLITBACK
 Wire Wire Line
-	10250 2450 10200 2450
+	8675 5075 9275 5075
 Wire Wire Line
-	8675 5075 10350 5075
-Wire Wire Line
-	8675 3125 10075 3125
-Wire Wire Line
-	10200 2450 10200 2525
-Connection ~ 10200 2450
-Wire Wire Line
-	10200 2450 10150 2450
-$Comp
-L Device:Jumper_NO_Small JP1
-U 1 1 63F65960
-P 10100 2525
-F 0 "JP1" H 10100 2710 50  0000 C CNN
-F 1 "UnifiedJumper" H 10100 2619 50  0000 C CNN
-F 2 "random-keyboard-parts:Jumper-UserFriendly" H 10100 2525 50  0001 C CNN
-F 3 "~" H 10100 2525 50  0001 C CNN
-	1    10100 2525
-	1    0    0    -1
-$EndComp
-$Comp
-L Device:Jumper_NO_Small JP2
-U 1 1 63F65CB6
-P 10300 2525
-F 0 "JP2" H 10300 2710 50  0000 C CNN
-F 1 "SplitJumper" H 10300 2619 50  0000 C CNN
-F 2 "random-keyboard-parts:Jumper-UserFriendly" H 10300 2525 50  0001 C CNN
-F 3 "~" H 10300 2525 50  0001 C CNN
-	1    10300 2525
-	1    0    0    -1
-$EndComp
-Connection ~ 10200 2525
-Wire Wire Line
-	10400 2525 10400 2750
-Wire Wire Line
-	10400 2750 10350 2750
-Wire Wire Line
-	10000 2525 10000 2750
-Wire Wire Line
-	10000 2750 10075 2750
-Wire Wire Line
-	10075 2950 10075 3125
-Connection ~ 10075 3125
-Wire Wire Line
-	10075 3125 11050 3125
-Wire Wire Line
-	10350 2950 10350 5075
-Connection ~ 10350 5075
-Wire Wire Line
-	10350 5075 11650 5075
+	8675 3125 9275 3125
 Wire Wire Line
 	12525 5325 12525 3375
 Connection ~ 12525 3375
+Connection ~ 9275 5075
+Connection ~ 9275 3125
+Wire Wire Line
+	9275 3125 11050 3125
+Wire Wire Line
+	9275 5075 11650 5075
 $EndSCHEMATC
